File: bkc40/bkc40.sch (KiCad schematic (older format))
At the start: 105 parts, among them J1 Conn_01x02, SW1 SW_Push, SW10 SW_Push, SW11 SW_Push, SW12 SW_Push, SW13 SW_Push, SW14 SW_Push, SW15 SW_Push, SW16 SW_Push, SW17 SW_Push, SW18 SW_Push, SW19 SW_Push, SW2 SW_Push, SW20 SW_Push, SW21 SW_Push, SW22 SW_Push, SW23 SW_Push, SW24 SW_Push, SW25 SW_Push, SW26 SW_Push, SW27 SW_Push, SW28 SW_Push, SW29 SW_Push, SW3 SW_Push, SW30 SW_Push, SW31 SW_Push, SW32 SW_Push, SW33 SW_Push, SW34 SW_Push, SW35 SW_Push, SW36 SW_Push, SW37 SW_Push, SW38 SW_Push, SW39 SW_Push, SW4 SW_Push, SW40 SW_Push, SW41 SW_Push, SW42 SW_Push, SW43 SW_Push, SW44 SW_Push, SW45 SW_Push, SW46 SW_Push, SW47 SW_Push, SW48 SW_Push, SW49 SW_Push, SW5 SW_Push, SW50 SW_Push, SW51 SW_Push, SW52 SW_Push, SW53 SW_Push, SW54 SW_Push, SW55 SW_Push, SW56 Rotary_Encoder_Switch, SW57 SW_Push, SW6 SW_Push, SW7 SW_Push, SW8 SW_Push, SW9 SW_Push, U1 ATmega32U4-AU, Y1 Crystal_GND24_Small

Commit message: v02
Parts:
- removed U1: ATmega32U4-AU, Package_QFP:TQFP-44_10x10mm_P0.8mm, symbol MCU_Microchip_ATmega:ATmega32U4-AU
- added U2: ATmega32U4-MU, Package_DFN_QFN:QFN-44-1EP_7x7mm_P0.5mm_EP5.2x5.2mm, symbol MCU_Microchip_ATmega:ATmega32U4-MU
Connections:
- net +5V: now also U2.14 (VCC), U2.2 (UVCC), U2.24 (AVCC), U2.34 (VCC), U2.44 (AVCC), U2.7 (VBUS)
- net COL00: now also U2.37 (PF6)
- net COL01: now also U2.20 (PD2)
- net COL02: now also U2.19 (PD1)
- net COL03: now also U2.18 (PD0)
- net COL04: now also U2.21 (PD3)
- net COL05: now also U2.25 (PD4)
- net COL06: now also U2.26 (PD6)
- net COL07: now also U2.27 (PD7)
- net COL08: now also U2.28 (PB4)
- net COL09: now also U2.29 (PB5)
- net COL10: now also U2.30 (PB6)
- net COL11: now also U2.31 (PC6)
- net COL12: now also U2.32 (PC7)
- net D+: now also U2.4 (D+)
- net D-: now also U2.3 (D-)
- net ENC_A: now also U2.38 (PF5)
- net ENC_B: now also U2.39 (PF4)
- net GND: now also U2.15 (GND), U2.23 (GND), U2.35 (GND), U2.43 (GND), U2.45 (GND), U2.5 (UGND)
- net ROW00: now also U2.41 (PF0)
- net ROW01: now also U2.1 (PE6)
- net ROW02: now also U2.36 (PF7)
- net ROW03: now also U2.40 (PF1)
- net at J1.2 (Pin_2), R1.2: now also U2.13 (~RESET)
- net at C8.1, Y1.3: now also U2.16 (XTAL2)
- net at C7.1, Y1.1: now also U2.17 (XTAL1)
- net at R4.2: now also U2.33 (~HWB~/PE2)
- net at C9.1: now also U2.6 (UCAP)
- no-connect marks 2 -> 3
Changed lines of the file:
@@
 	21850 2900 21850 3350
-$Comp
-L MCU_Microchip_ATmega:ATmega32U4-AU U1
-U 1 1 621CC68E
-P 3350 12950
-F 0 "U1" H 3350 11061 50  0000 C CNN
-F 1 "ATmega32U4-AU" H 3350 10970 50  0000 C CNN
-F 2 "Package_QFP:TQFP-44_10x10mm_P0.8mm" H 3350 12950 50  0001 C CIN
-F 3 "http://ww1.microchip.com/downloads/en/DeviceDoc/Atmel-7766-8-bit-AVR-ATmega16U4-32U4_Datasheet.pdf" H 3350 12950 50  0001 C CNN
-	1    3350 12950
-	1    0    0    -1
-$EndComp
 $Comp
 L power:+5V #PWR0101
@@
 	1    0    0    -1
 $EndComp
-Wire Wire Line
-	3600 11150 3450 11150
-Connection ~ 3350 11150
-Wire Wire Line
-	3350 11150 3250 11150
-Connection ~ 3450 11150
-Wire Wire Line
-	3450 11150 3350 11150
 $Comp
 L power:GND #PWR0102
@@
 	1    0    0    -1
 $EndComp
-Wire Wire Line
-	2850 14750 3250 14750
-Connection ~ 3250 14750
-Wire Wire Line
-	3250 14750 3350 14750
 $Comp
 L Connector_Generic:Conn_01x02 J1
@@
 Wire Wire Line
 	7350 10850 7100 10850
+Text GLabel 3950 12050 2    50   Input ~ 0
+COL10
+Text GLabel 3950 11950 2    50   Input ~ 0
+COL09
+Text GLabel 3950 11850 2    50   Input ~ 0
+COL08
+Text GLabel 3950 13350 2    50   Input ~ 0
+COL07
+Text GLabel 3950 13250 2    50   Input ~ 0
+COL06
+Text GLabel 3950 13050 2    50   Input ~ 0
+COL05
+Text GLabel 3950 12950 2    50   Input ~ 0
+COL04
+Text GLabel 3950 12650 2    50   Input ~ 0
+COL03
+Text GLabel 3950 12750 2    50   Input ~ 0
+COL02
+Text GLabel 3950 12850 2    50   Input ~ 0
+COL01
+Text GLabel 3950 14250 2    50   Input ~ 0
+COL00
+Text GLabel 3950 13950 2    50   Input ~ 0
+ROW03
+Text GLabel 3950 12450 2    50   Input ~ 0
+COL12
 Text GLabel 3950 13850 2    50   Input ~ 0
-COL10
-Text GLabel 3950 13950 2    50   Input ~ 0
-COL09
-Text GLabel 3950 14050 2    50   Input ~ 0
-COL08
-Text GLabel 3950 14150 2    50   Input ~ 0
-COL07
-Text GLabel 3950 14250 2    50   Input ~ 0
-COL06
+ROW00
+Wire Wire Line
+	21450 3350 21450 4950
+Text GLabel 3950 13650 2    50   Input ~ 0
+ROW01
 Text GLabel 3950 14350 2    50   Input ~ 0
-COL05
-Text GLabel 3950 12450 2    50   Input ~ 0
-COL04
-Text GLabel 3950 12350 2    50   Input ~ 0
-COL03
-Text GLabel 3950 12050 2    50   Input ~ 0
-COL02
-Text GLabel 3950 11950 2    50   Input ~ 0
-COL01
-Text GLabel 3950 11850 2    50   Input ~ 0
-COL00
-Text GLabel 3950 13350 2    50   Input ~ 0
-ROW03
-Text GLabel 3950 13250 2    50   Input ~ 0
-COL12
-Text GLabel 3950 13050 2    50   Input ~ 0
-ROW00
-Wire Wire Line
-	21450 3350 21450 4950
-Text GLabel 3950 13150 2    50   Input ~ 0
-ROW01
-Text GLabel 3950 12950 2    50   Input ~ 0
 ROW02
 Wire Notes Line
@@
 Wire Wire Line
 	10850 14950 11300 14950
-Text GLabel 3950 12650 2    50   Input ~ 0
+Text GLabel 3950 14150 2    50   Input ~ 0
 ENC_A
-Text GLabel 3950 12750 2    50   Input ~ 0
+Text GLabel 3950 14050 2    50   Input ~ 0
 ENC_B
 Wire Notes Line
@@
 Text Notes 11800 15500 2    118  Italic 24
 ROTARY ENCODER
+Wire Wire Line
+	3250 11150 3350 11150
+Wire Wire Line
+	2850 14750 3250 14750
+Connection ~ 3350 11150
+Wire Wire Line
+	3350 14750 3250 14750
+Connection ~ 3250 14750
+Connection ~ 3450 11150
+Wire Wire Line
+	3450 11150 3600 11150
+Wire Wire Line
+	3350 11150 3450 11150
+$Comp
+L MCU_Microchip_ATmega:ATmega32U4-MU U2
+U 1 1 612D3612
+P 3350 12950
+F 0 "U2" H 3350 11061 50  0000 C CNN
+F 1 "ATmega32U4-MU" H 3350 10970 50  0000 C CNN
+F 2 "Package_DFN_QFN:QFN-44-1EP_7x7mm_P0.5mm_EP5.2x5.2mm" H 3350 12950 50  0001 C CIN
+F 3 "http://ww1.microchip.com/downloads/en/DeviceDoc/Atmel-7766-8-bit-AVR-ATmega16U4-32U4_Datasheet.pdf" H 3350 12950 50  0001 C CNN
+	1    3350 12950
+	1    0    0    -1
+$EndComp
+NoConn ~ 2750 12050
+Text GLabel 3950 12350 2    50   Input ~ 0
+COL11
 $EndSCHEMATC

Commit message: update cc pins
Parts:
- added SW58: SW_Push, MX_Only:MXOnly-1.25U-NoLED, symbol Switch:SW_Push
- Y1: value Crystal_GND24_Small -> 16Mhz
Connections:
- net COL00: now also SW58.1
- net GND: now also USB1.1 (GND), USB1.12 (GND)
- net at D8.2 (A), SW16.2: now also SW58.2
- net at R5.2: now also USB1.4 (CC1); no longer USB1.1 (GND)
- net at USB1.10 (CC2): now also R6.2
- no-connect marks 3 -> 4
Changed lines of the file:
@@
 	7050 5350 7050 6200
 Wire Wire Line
-	7050 3700 7050 4950
+	7050 3700 7050 4050
 Wire Wire Line
 	7450 4950 7450 4600
@@
 P 2500 11750
 F 0 "Y1" V 2454 11894 50  0000 L CNN
-F 1 "Crystal_GND24_Small" V 2545 11894 50  0000 L CNN
+F 1 "16Mhz" V 2545 11894 50  0000 L CNN
 F 2 "Crystal:Crystal_SMD_3225-4Pin_3.2x2.5mm" H 2500 11750 50  0001 C CNN
 F 3 "~" H 2500 11750 50  0001 C CNN
@@
 Wire Wire Line
 	8300 12700 7950 12700
-Wire Wire Line
-	7950 12700 7550 12700
 Connection ~ 7950 12700
 $Comp
@@
 $EndComp
 Wire Wire Line
-	7250 12600 7450 12600
-Wire Wire Line
-	7450 12600 7450 14400
-Wire Wire Line
-	7450 14400 8800 14400
-Wire Wire Line
 	8800 14400 8800 14250
-Wire Wire Line
-	7250 13700 7350 13700
-Wire Wire Line
-	7350 13700 7350 14550
-Wire Wire Line
-	7350 14550 8800 14550
 Wire Wire Line
 	9000 14550 9000 14250
@@
 Wire Wire Line
 	9000 14000 9000 14250
-Wire Wire Line
-	7250 13600 7550 13600
-Wire Wire Line
-	7550 13600 7550 12700
-Connection ~ 7550 12700
-Wire Wire Line
-	7550 12700 7250 12700
 $Comp
 L Device:R_Small R7
@@
 Text GLabel 3950 12350 2    50   Input ~ 0
 COL11
+$Comp
+L Switch:SW_Push SW58
+U 1 1 61417C4D
+P 7250 4050
+F 0 "SW58" H 7250 4335 50  0000 C CNN
+F 1 "SW_Push" H 7250 4244 50  0000 C CNN
+F 2 "MX_Only:MXOnly-1.25U-NoLED" H 7250 4250 50  0001 C CNN
+F 3 "~" H 7250 4250 50  0001 C CNN
+	1    7250 4050
+	1    0    0    -1
+$EndComp
+Connection ~ 7050 4050
+Wire Wire Line
+	7050 4050 7050 4950
+Wire Wire Line
+	7450 4050 7450 3700
+Connection ~ 7450 3700
+NoConn ~ 16550 -700
+Wire Wire Line
+	7250 12600 7400 12600
+Wire Wire Line
+	7400 12600 7400 13700
+Wire Wire Line
+	7250 13700 7400 13700
+Wire Wire Line
+	7250 12700 7750 12700
+Wire Wire Line
+	7750 13600 7750 12700
+Wire Wire Line
+	7250 13600 7750 13600
+Connection ~ 7750 12700
+Wire Wire Line
+	7750 12700 7950 12700
+$Comp
+L power:GND #PWR0119
+U 1 1 6166AADD
+P 7400 13700
+F 0 "#PWR0119" H 7400 13450 50  0001 C CNN
+F 1 "GND" H 7405 13527 50  0000 C CNN
+F 2 "" H 7400 13700 50  0001 C CNN
+F 3 "" H 7400 13700 50  0001 C CNN
+	1    7400 13700
+	1    0    0    -1
+$EndComp
+Connection ~ 7400 13700
+Wire Wire Line
+	7250 12900 7650 12900
+Wire Wire Line
+	7650 12900 7650 14400
+Wire Wire Line
+	7650 14400 8800 14400
+Wire Wire Line
+	7250 13500 7550 13500
+Wire Wire Line
+	7550 13500 7550 14550
+Wire Wire Line
+	7550 14550 8800 14550
 $EndSCHEMATC
